File: DuelTank/DuelTank.kicad_pcb (KiCad board)
At the start: 2 copper layers, 114.3 x 88.9 mm, 50 parts, among them J1 AudioJack, J2 Speaker, J3 UART1, J4 Pot, J6 GND, J7 DACOUT, SW1 UP, SW2 LEFT, SW3 DOWN, SW4 RGHT, U1 Adafruit ST7735R, U2 LP-MSPM0G3507, U3 MCP34119P, U4 HiLetGo_ST7735R, U5 ULN2003B, U6 TSOP31438

Commit message: hardware done
Parts:
- removed D4: LED, ECE319K:LED_D5.0mm
- removed J1: AudioJack, ECE319K:Jack_3.5mm_CUI_SJ1-3523N_Horizontal
- removed R2, R3: 220, ECE319K:R_Axial_DIN0204_L3.6mm_D1.6mm_P7.62mm_Horizontal
- removed U1: Adafruit ST7735R, ECE319K:adafruit_st7735r
- removed U6: TSOP31438, ECE319K:TSOP31438
- added C5: 0.1uF, ECE319K:C_Axial_200mil, F.Cu at (131.4, 101.0)
- added C6: 0.1uF, ECE319K:C_Axial_200mil, F.Cu at (164.3, 42.0)
- added C7: 0.1uF, ECE319K:C_Axial_200mil, F.Cu at (157.2, 101.3)
- added D10: GREEN_LED4, ECE319K:LED_D5.0mm, F.Cu at (189.5, 94.0)
- added D5: GREEN_LED3, ECE319K:LED_D5.0mm, F.Cu at (189.5, 85.7)
- added D8: YellowLED_TX, ECE319K:LED_D5.0mm, F.Cu at (189.5, 52.7)
- added D9: YellowLED_RX, ECE319K:LED_D5.0mm, F.Cu at (189.5, 61.0)
- added G***: LOGO, images:fire, F.Cu at (120.1, 106.5)
- added G***: LOGO, images:arrow, F.Cu at (149.6, 109.2)
- added G***: LOGO, images:shield, F.Cu at (96.4, 108.9)
- added G***: LOGO, images:arrow, F.Cu at (180.6, 108.8)
- added J5: 1053131105, nanofit_1x5:CONN_SD-105313-100_05_MOL, F.Cu at (91.3, 44.4)
- added R19: 1.5k, ECE319K:R_Axial_DIN0204_L3.6mm_D1.6mm_P7.62mm_Horizontal, F.Cu at (121.5, 24.5)
- added R20: 10k, ECE319K:R_Axial_DIN0204_L3.6mm_D1.6mm_P7.62mm_Horizontal, F.Cu at (144.5, 33.0)
- added R21: 300, ECE319K:R_Axial_DIN0204_L3.6mm_D1.6mm_P7.62mm_Horizontal, F.Cu at (179.6, 52.4)
- added R22: 300, ECE319K:R_Axial_DIN0204_L3.6mm_D1.6mm_P7.62mm_Horizontal, F.Cu at (179.6, 54.9)
- added R23: 300, ECE319K:R_Axial_DIN0204_L3.6mm_D1.6mm_P7.62mm_Horizontal, F.Cu at (179.6, 65.0)
- added TP10: Divider1, TestPoint:TestPoint_Pad_D2.0mm, B.Cu at (111.3, 33.8)
- added TP11: Divider2, TestPoint:TestPoint_Pad_D2.0mm, B.Cu at (116.8, 33.8)
- added TP12: Divider3, TestPoint:TestPoint_Pad_D2.0mm, B.Cu at (121.5, 38.8)
- added TP13: Divider4, TestPoint:TestPoint_Pad_D2.0mm, B.Cu at (126.6, 33.8)
- added TP14: Divider5, TestPoint:TestPoint_Pad_D2.0mm, B.Cu at (131.4, 33.8)
- added TP16: SlidePot, TestPoint:TestPoint_Pad_D2.0mm, B.Cu at (95.2, 68.9)
- added TP17: DACOUT, TestPoint:TestPoint_Pad_D2.0mm, B.Cu at (115.5, 24.9)
- added TP2: Left_SW, TestPoint:TestPoint_Pad_D2.0mm, B.Cu at (151.4, 109.1)
- added TP3: Shield_SW, TestPoint:TestPoint_Pad_D2.0mm, B.Cu at (96.7, 109.1)
- added TP4: Right_SW, TestPoint:TestPoint_Pad_D2.0mm, B.Cu at (178.7, 109.1)
- added TP5: Fire_SW, TestPoint:TestPoint_Pad_D2.0mm, B.Cu at (124.0, 109.1)
- D1: value LED -> PWR_RED
- D2: value LED -> GREEN_LED1
- D3: value LED -> GREEN_LED2
- H1, H2, H3, H4: value ~ -> M.3; footprint ECE319K:MountingHole_4_40 -> MountingHole:MountingHole_3.2mm_M3_Pad_TopBottom
- J3: value UART1 -> 1053131105; footprint ECE319K:PinHeader_1x03_P2.54mm_Vertical -> nanofit_1x5:CONN_SD-105313-100_05_MOL
- R1: value 220 -> 300
- R10, R11, R9: value 12k -> 1.5k
- R16: value 20k -> 12k
- R17: value 10k -> 12k
- R18: value 220 -> 12k
- R4, R5, R6: value 1.5k -> 300
- R7: value 1.5k -> 20k
- SW1: value UP -> Shield
- SW2: value LEFT -> Fire
- SW3: value DOWN -> Left
- SW4: value RGHT -> Right
- moved H3 167.7 mm to (192.0, 27.0)
- moved U5 163.0 mm to (172.0, 75.2)
- moved C2 147.0 mm to (156.0, 38.9), turned to 180 degrees
- moved SW4 143.4 mm to (175.5, 106.9)
- moved C1 138.8 mm to (142.6, 38.9)
- moved J2 136.3 mm to (161.5, 31.5)
- moved U3 135.6 mm to (155.3, 25.3)
- moved R14 133.7 mm to (161.1, 99.9), turned to 0 degrees
- moved R15 126.9 mm to (161.1, 97.5), turned to 0 degrees
- moved H4 123.4 mm to (84.0, 27.0)
- moved U4 116.2 mm to (139.6, 69.8), turned to 90 degrees
- moved C4 116.1 mm to (136.8, 101.0), turned to 90 degrees
- moved R6 112.7 mm to (179.6, 62.7), turned to 180 degrees
- moved R18 111.6 mm to (131.7, 29.2), turned to -90 degrees
- moved C3 109.2 mm to (138.9, 26.5)
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Connections:
- C1 pad 1: unconnected-(C1-Pad1) -> Net-(U3-FC1)
- C1 pad 2: unconnected-(C1-Pad2) -> GND
- C2 pad 1: unconnected-(C2-Pad1) -> Net-(U3-FC2)
- C2 pad 2: unconnected-(C2-Pad2) -> GND
- C3 pad 1: unconnected-(C3-Pad1) -> DACOUT
- C3 pad 2: unconnected-(C3-Pad2) -> Net-(C3-Pad2)
- C4 pad 1: unconnected-(C4-Pad1) -> GND
- C4 pad 2: unconnected-(C4-Pad2) -> PB17
- D1 pad 1: unconnected-(D1-K-Pad1) -> GND
- D1 pad 2: unconnected-(D1-A-Pad2) -> Net-(D1-A)
- D2 pad 1: unconnected-(D2-K-Pad1) -> Net-(D2-K)
- D2 pad 2: unconnected-(D2-A-Pad2) -> +5V
- D3 pad 1: unconnected-(D3-K-Pad1) -> Net-(D3-K)
- D3 pad 2: unconnected-(D3-A-Pad2) -> +5V
- H1 pad 1: unconnected-(H1-Hole-Pad1) -> (no net)
- H2 pad 1: unconnected-(H2-Hole-Pad1) -> (no net)
- H3 pad 1: unconnected-(H3-Hole-Pad1) -> (no net)
- H4 pad 1: unconnected-(H4-Hole-Pad1) -> (no net)
- J2 pad 1: unconnected-(J2-Pad1) -> Net-(U3-VO1)
- J2 pad 2: unconnected-(J2-Pad2) -> Net-(U3-VO2)
- J3 pad 2: PA8 -> PA31
- J3 pad 3: PA22 -> PA17
- J4 pad 1: unconnected-(J4-A-Pad1) -> PB18
- J4 pad 2: unconnected-(J4-B-Pad2) -> PB18
- J7 pad 1: unconnected-(J7-A-Pad1) -> DACOUT
- J7 pad 2: unconnected-(J7-B-Pad2) -> DACOUT
- JP1 pad 1: unconnected-(JP1-A-Pad1) -> PB20
- JP1 pad 3: unconnected-(JP1-B-Pad3) -> PB20
- R1 pad 1: unconnected-(R1-Pad1) -> +5V
- R1 pad 2: unconnected-(R1-Pad2) -> Net-(D1-A)
- R10 pad 1: unconnected-(R10-Pad1) -> DACOUT
- R10 pad 2: unconnected-(R10-Pad2) -> PB0
- R11 pad 1: unconnected-(R11-Pad1) -> DACOUT
- R11 pad 2: unconnected-(R11-Pad2) -> PB0
- R12 pad 1: unconnected-(R12-Pad1) -> PB12
- R12 pad 2: unconnected-(R12-Pad2) -> GND
- R13 pad 1: unconnected-(R13-Pad1) -> PB17
- R13 pad 2: unconnected-(R13-Pad2) -> GND
- R14 pad 1: unconnected-(R14-Pad1) -> PB16
- R14 pad 2: unconnected-(R14-Pad2) -> GND
- R15 pad 1: unconnected-(R15-Pad1) -> PA27
- R15 pad 2: unconnected-(R15-Pad2) -> GND
- R16 pad 1: unconnected-(R16-Pad1) -> DACOUT
- R16 pad 2: unconnected-(R16-Pad2) -> PB3
- R17 pad 1: unconnected-(R17-Pad1) -> DACOUT
- R17 pad 2: unconnected-(R17-Pad2) -> PB3
- R18 pad 1: unconnected-(R18-Pad1) -> DACOUT
- R18 pad 2: unconnected-(R18-Pad2) -> PB4
- R4 pad 1: unconnected-(R4-Pad1) -> Net-(D2-K)
- R4 pad 2: unconnected-(R4-Pad2) -> Net-(U5-3C)
- R5 pad 1: unconnected-(R5-Pad1) -> Net-(D3-K)
- R5 pad 2: unconnected-(R5-Pad2) -> Net-(U5-4C)
- R6 pad 1: unconnected-(R6-Pad1) -> Net-(D5-K)
- R6 pad 2: unconnected-(R6-Pad2) -> Net-(U5-5C)
- R7 pad 1: unconnected-(R7-Pad1) -> Net-(U3-VIN)
- R7 pad 2: unconnected-(R7-Pad2) -> Net-(C3-Pad2)
- R8 pad 1: unconnected-(R8-Pad1) -> Net-(R19-Pad2)
- R8 pad 2: unconnected-(R8-Pad2) -> PB2
- R9 pad 1: unconnected-(R9-Pad1) -> DACOUT
- R9 pad 2: unconnected-(R9-Pad2) -> PB1
- RV1 pad 1: unconnected-(RV1-Pad1) -> GND
- RV1 pad 2: unconnected-(RV1-Pad2) -> PB18
- RV1 pad 3: unconnected-(RV1-Pad3) -> +3V3
- SW1 pad 1: unconnected-(SW1-Pad1) -> PB12
- SW1 pad 2: unconnected-(SW1-Pad2) -> +3V3
- SW2 pad 1: unconnected-(SW2-Pad1) -> PB17
- SW2 pad 2: unconnected-(SW2-Pad2) -> +3V3
- SW3 pad 1: unconnected-(SW3-Pad1) -> PB16
- SW3 pad 2: unconnected-(SW3-Pad2) -> +3V3
- SW4 pad 1: unconnected-(SW4-Pad1) -> PA27
- SW4 pad 2: unconnected-(SW4-Pad2) -> +3V3
- U3 pad 2: unconnected-(U3-FC2-Pad2) -> Net-(U3-FC2)
- U3 pad 3: unconnected-(U3-FC1-Pad3) -> Net-(U3-FC1)
- U3 pad 4: unconnected-(U3-VIN-Pad4) -> Net-(U3-VIN)
- U3 pad 5: unconnected-(U3-VO1-Pad5) -> Net-(U3-VO1)
- U3 pad 6: unconnected-(U3-Vcc-Pad6) -> +5V
- U3 pad 7: unconnected-(U3-GND-Pad7) -> GND
- U3 pad 8: unconnected-(U3-VO2-Pad8) -> Net-(U3-VO2)
- U5 pad 1: unconnected-(U5-1B-Pad1) -> PA15
- U5 pad 11: unconnected-(U5-6C-Pad11) -> Net-(U5-6C)
- U5 pad 12: unconnected-(U5-5C-Pad12) -> Net-(U5-5C)
- U5 pad 13: unconnected-(U5-4C-Pad13) -> Net-(U5-4C)
- U5 pad 14: unconnected-(U5-3C-Pad14) -> Net-(U5-3C)
- U5 pad 15: unconnected-(U5-2C-Pad15) -> LED_RX
- U5 pad 16: unconnected-(U5-1C-Pad16) -> LED_TX
- U5 pad 2: unconnected-(U5-2B-Pad2) -> PA16
- U5 pad 3: unconnected-(U5-3B-Pad3) -> PA24
- U5 pad 4: unconnected-(U5-4B-Pad4) -> PA18
- U5 pad 5: unconnected-(U5-5B-Pad5) -> PB19
- U5 pad 6: unconnected-(U5-6B-Pad6) -> PB13
- U5 pad 8: unconnected-(U5-E-Pad8) -> GND
Routing:
- net PA31: track 0.00 -> 177.2 mm, vias 0 -> 2
- net +5V: track 0.00 -> 108.8 mm
- net PA17: track 0.00 -> 108.7 mm, vias 0 -> 4
- net PA27: track 0.00 -> 102.1 mm, vias 0 -> 1
- net PA8: track 0.00 -> 100.8 mm
- net PB18: track 0.00 -> 99.5 mm, vias 0 -> 6
- net PA22: track 0.00 -> 98.4 mm
- net PB0: track 0.00 -> 91.5 mm, vias 0 -> 2
- net PB4: track 0.00 -> 71.3 mm, vias 0 -> 1
- net PB1: track 0.00 -> 67.0 mm, vias 0 -> 1
- net PA12: track 0.00 -> 63.0 mm
- net GND: track 0.00 -> 59.8 mm, vias 0 -> 19
- net PB12: track 0.00 -> 59.5 mm
- net PB19: track 0.00 -> 57.6 mm
- net PB8: track 0.00 -> 57.2 mm
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- added copper zone on F.Cu, net +3V3
- added copper zone on F.Cu, net +5V
- added copper zone on F.Cu, net DACOUT
- added copper zone on B.Cu, net GND
Other:
- board size 114.3 x 88.9 mm -> 118 x 100 mm
- board text added: "0.75"
- board text added: "1.5"
- board text added: "12.0"
- board text added: "3.0"
- board text added: "6.0"
- board text added: "LED_RX"
- board text added: "LED_TX"
- board text added: "Made by Sathvik Yechuri :)"
- board text added: "R23"
- board text added: "SLIDE POT"
- board text added: "Sathvik Yechuri ECE319H - Final Project Spring 2026"
- board text added: "XLED_1"
- board text added: "XLED_2"
- board text added: "XLED_3"
- board text added: "XLED_4"
- board text removed: "DACOUT"
- board text removed: "ECE319K PCB camp Spring 2026"
- board text removed: "GND"
- board text removed: "POT"
- board text removed: "TExaS"
- board text removed: "U1Rx"
- board text removed: "U1Tx"
- board text removed: "Your names"

Commit message: board ordered!
Parts:
- removed U4: HiLetGo_ST7735R, ECE319K:hiletgo_st7735r
- added J8: Conn_01x08, Connector_PinHeader_2.54mm:PinHeader_1x08_P2.54mm_Vertical, F.Cu at (115.2, 78.5)
Routing:
- net PA12: track 63.0 -> 0.00 mm
- net PB7: track 55.3 -> 0.00 mm
- net GND: track 59.8 -> 81.8 mm, vias 19 -> 27
- net PB8: track 57.2 -> 43.9 mm, vias 0 -> 1
- net PB6: track 53.6 -> 43.6 mm, vias 1 -> 0
- net PA13: track 56.4 -> 49.4 mm, vias 0 -> 1
- net PB9: track 52.4 -> 46.2 mm, vias 3 -> 5
- net PB15: track 33.8 -> 32.0 mm
- net PB1: track 67.0 -> 65.5 mm
- net PA31: track 177.2 -> 177.9 mm
Other:
- board text added: "FIRE!"
- board text added: "LEFT"
- board text added: "RIGHT"
- board text added: "SHIELD"
