File: DuelTank/DuelTank.kicad_sch (KiCad schematic)
At the start: 45 parts, among them J1 AudioJack, J2 Speaker, J4 Pot, J6 GND, J7 DACOUT, SW1 Shield, SW2 Fire, SW3 Left, SW4 Right, U2 LP-MSPM0G3507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

Commit message: yay
Parts:
- removed D?: GREEN_LED3, ECE319K:LED_D5.0mm, symbol ECE319K:LED
- removed D?: GREEN_LED4, ECE319K:LED_D5.0mm, symbol ECE319K:LED
- added D5: GREEN_LED3, ECE319K:LED_D5.0mm, symbol ECE319K:LED
- added D6: GREEN_LED4, ECE319K:LED_D5.0mm, symbol ECE319K:LED
- added D7: GREEN_LED5, ECE319K:LED_D5.0mm, symbol ECE319K:LED
- added D8: YellowLED_TX, ECE319K:LED_D5.0mm, symbol ECE319K:LED
- added D9: YellowLED_RX, ECE319K:LED_D5.0mm, symbol ECE319K:LED
- added H1, H2, H3, H4: M.3, MountingHole:MountingHole_3.2mm_M3_Pad_TopBottom, symbol Mechanical:MountingHole
- added J3: 1053131204, nanofit_1x4:nanofit_1x4, symbol nanofit_1x4:1053131204
- added R21, R22, R6: 300, ECE319K:R_Axial_DIN0204_L3.6mm_D1.6mm_P7.62mm_Horizontal, symbol ECE319K:R_0.125W
- added TP10: Divider1, TestPoint:TestPoint_Pad_D2.0mm, symbol Connector:TestPoint
- added TP11: Divider2, TestPoint:TestPoint_Pad_D2.0mm, symbol Connector:TestPoint
- added TP12: Divider3, TestPoint:TestPoint_Pad_D2.0mm, symbol Connector:TestPoint
- added TP13: Divider4, TestPoint:TestPoint_Pad_D2.0mm, symbol Connector:TestPoint
- added TP14: Divider5, TestPoint:TestPoint_Pad_D2.0mm, symbol Connector:TestPoint
- added TP15, TP6: LED2, TestPoint:TestPoint_Pad_D2.0mm, symbol Connector:TestPoint
- added TP16: SlidePot, TestPoint:TestPoint_Pad_D2.0mm, symbol Connector:TestPoint
- added TP17: DACOUT, TestPoint:TestPoint_Pad_D2.0mm, symbol Connector:TestPoint
- added TP2: Left_SW, TestPoint:TestPoint_Pad_D2.0mm, symbol Connector:TestPoint
- added TP3: Shield_SW, TestPoint:TestPoint_Pad_D2.0mm, symbol Connector:TestPoint
- added TP4: Right_SW, TestPoint:TestPoint_Pad_D2.0mm, symbol Connector:TestPoint
- added TP5: Fire_SW, TestPoint:TestPoint_Pad_D2.0mm, symbol Connector:TestPoint
- added TP7: LED1, TestPoint:TestPoint_Pad_D2.0mm, symbol Connector:TestPoint
- added TP8: LED4, TestPoint:TestPoint_Pad_D2.0mm, symbol Connector:TestPoint
- added TP9: LED3, TestPoint:TestPoint_Pad_D2.0mm, symbol Connector:TestPoint
- C3: value 0.1F -> 0.1uF
- R20: renamed from R?; value 75k -> 10k
- R7: renamed from R?; value 3k -> 20k
- gave numbers to parts that had none: 12
Connections:
- net +5V: now also D5.1 (K), D6.1 (K), D7.1 (K), D8.1 (K), D9.1 (K)
- net DACOUT: now also TP17.1
- net GND: now also J3.4, TP2.1, TP3.1, TP4.1, TP5.1
- net PA16: now also TP8.1
- net PA17: now also J3.3
- net PA18: now also TP6.1
- net PA22: now also U5.6 (6B), J3.1
- net PA24: now also TP9.1
- net PA28: now also U5.5 (5B), TP15.1
- net PA8: now also U5.7 (7B), J3.2
- net PB0: now also TP10.1
- net PB1: now also TP11.1
- net PB18: now also TP16.1
- net PB19: now also TP7.1
- net PB2: now also TP12.1
- net PB3: now also TP13.1
- net PB4: now also TP14.1
- net at R4.1: now also D5.2 (A)
- net at R5.1: now also D6.2 (A)
- net LED_RX: now reaches U5.10 (7C)
- net LED_RX: now also R22.2
- net LED_TX: now reaches U5.11 (6C)
- net LED_TX: now also R21.2
- net at U5.12 (5C): now also R6.2
- new net: D7.2 (A), R6.1
- new net: D9.2 (A), R22.1
- new net: D8.2 (A), R21.1
- no-connect marks 8 -> 11
Other:
- note added: "Battle_Rd_t"
- note added: "Made with sweat and tears by Sathvik Y :) (no blood yet)"
- note added: "Test points"
- note added: "UART Status"
- note removed: "Bat_Rd_t"
- moved on the sheet: D4, J1, U6

Commit message: hardware done
Parts:
- removed D6: GREEN_LED4, ECE319K:LED_D5.0mm, symbol ECE319K:LED
- removed D7: GREEN_LED5, ECE319K:LED_D5.0mm, symbol ECE319K:LED
- removed J3: 1053131204, nanofit_1x4:nanofit_1x4, symbol nanofit_1x4:1053131204
- removed R2, R3: 300, ECE319K:R_Axial_DIN0204_L3.6mm_D1.6mm_P7.62mm_Horizontal, symbol ECE319K:R_0.125W
- removed TP15, TP6: LED2, TestPoint:TestPoint_Pad_D2.0mm, symbol Connector:TestPoint
- removed TP7: LED1, TestPoint:TestPoint_Pad_D2.0mm, symbol Connector:TestPoint
- removed TP8: LED4, TestPoint:TestPoint_Pad_D2.0mm, symbol Connector:TestPoint
- removed TP9: LED3, TestPoint:TestPoint_Pad_D2.0mm, symbol Connector:TestPoint
- added C4, C5, C6, C7: 0.1uF, ECE319K:C_Axial_200mil, symbol ECE319K:C
- added D10: GREEN_LED4, ECE319K:LED_D5.0mm, symbol ECE319K:LED
- added J3, J5: 1053131105, nanofit_1x5:CONN_SD-105313-100_05_MOL, symbol nanofit_1x5:1053131105
- added R23: 300, ECE319K:R_Axial_DIN0204_L3.6mm_D1.6mm_P7.62mm_Horizontal, symbol ECE319K:R_0.125W
Connections:
- net +3V3: now also SW1.2, SW2.2, SW3.2, SW4.2; no longer R12.1, R13.1, R14.1, R15.1
- net +5V: now also D2.2 (A), D3.2 (A), D5.2 (A), D8.2 (A), D9.2 (A), D10.2 (A); no longer D2.1 (K), D3.1 (K), D5.1 (K), D8.1 (K), D9.1 (K)
- net DACOUT: no longer JP1.1 (A)
- net GND: now also R12.2, R13.2, R14.2, R15.2, C4.1, C5.1, C6.1, C7.1, J3.1, J5.5; no longer SW1.1, SW2.1, SW3.1, SW4.1, TP2.1, TP3.1, TP4.1, TP5.1, U2.J1_3 (PA9/PB23), U2.J1_5 (PA26), U2.J1_6 (PB24), U2.J1_8 (PA27)
- net LED_RX: now also U5.15 (2C); no longer U5.10 (7C)
- net LED_TX: now also U5.16 (1C); no longer U5.11 (6C)
- net PA15: now also U5.1 (1B)
- net PA16: now also U5.2 (2B); no longer U5.4 (4B)
- net PA17: now also J3.3, J5.3
- net PA18: now also U5.4 (4B); no longer U5.2 (2B)
- net PA22: now also J3.5, J5.1; no longer U5.6 (6B)
- net PA28: no longer U5.5 (5B)
- net PA31: now also J3.2, J5.4
- net PA8: now also J3.4, J5.2; no longer U5.7 (7B)
- net PB12: now also R12.1, SW1.1, TP3.1, C5.2
- net PB13: now also U5.6 (6B)
- net PB16: now also R14.1, SW3.1, TP2.1, C7.2
- net PB17: now also R13.1, SW2.1, TP5.1, C4.2
- net PB18: no longer JP1.3 (B)
- net PB19: now also U5.5 (5B); no longer U5.1 (1B)
- net PB20: now also JP1.1 (A), JP1.3 (B)
- net at R6.1: now also D5.1 (K)
- net at R22.1: now also D9.1 (K); no longer D9.2 (A)
- net at R5.1: now also D3.1 (K)
- net at R21.1: now also D8.1 (K); no longer D8.2 (A)
- net at R4.1: now also D2.1 (K); no longer D5.2 (A)
- new net: D10.1 (K), R23.1
- new net: R23.2, U5.11 (6C)
- new net PA26: U2.J1_5 (PA26)
- new net PA27: C6.2, R15.1, SW4.1, TP4.1, U2.J1_8 (PA27)
- new net PB23: U2.J1_3 (PA9/PB23)
- new net PB24: U2.J1_6 (PB24)
- no-connect marks 11 -> 13
Other:
- note added: "Battle_Rd_t_1"
- note added: "Battle_Rd_t_2"
- note added: "UART Comms TX/RX"
- note removed: "Battle_Rd_t"
- note removed: "UART Comms"
- moved on the sheet: D1, D2, D3, D5, D8, D9, H1, H2, H3, H4, R1, R12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

Commit message: board ordered!
Parts:
- removed U4: HiLetGo_ST7735R, ECE319K:hiletgo_st7735r, symbol ECE319K:HiLetGo_ST7735R
- added J8: Conn_01x08, Connector_PinHeader_2.54mm:PinHeader_1x08_P2.54mm_Vertical, symbol Connector_Generic:Conn_01x08
Connections:
- net +3V3: now also J8.6 (Pin_6), J8.7 (Pin_7)
- net GND: now also J8.8 (Pin_8)
- net PA13: now also J8.3 (Pin_3)
- net PB15: now also J8.1 (Pin_1)
- net PB6: now also J8.2 (Pin_2)
- net PB8: now also J8.4 (Pin_4)
- net PB9: now also J8.5 (Pin_5)
- no-connect marks 13 -> 14
Other:
- moved on the sheet: D4, D8, D9, H1, H2, H3, H4, J1, J3, J5, JP1, R21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
